File: KiCad/BetaBoard.sch (KiCad schematic (older format))
At the start: 42 parts

Commit message: +Add per channel decoder. *Spread out the clock drivers more evenly. *Misc tidy up.
Parts:
- added J?: RJ45, symbol RJ45
- added U? (x2): 74HC154, symbol 74LS154
- U?: symbol SP485R -> SP485R-RESCUE-BetaBoard
Connections:
- net CLK2: no longer J?.3
- net CLK3: now also J?.3; no longer J?.3, J?.3
- net CLK4: now also J?.3, J?.3
- net DATA00: now also U?.1 (S0)
- net DATA01: now also U?.2 (S1)
- net DATA02: now also U?.3 (S2)
- net DATA03: now also U?.4 (S3)
- net DATA04: now also U?.5 (S4)
- net DATA05: now also U?.6 (S5)
- net DATA06: now also U?.7 (S6)
- net DATA07: now also U?.8 (S7)
- net DATA08: now also U?.9 (S8)
- net DATA09: now also U?.10 (S9)
- net DATA10: now also U?.11 (S10)
- net DATA11: now also U?.13 (S11)
- net DATA12: now also U?.14 (S12)
- net DATA13: now also U?.15 (S13)
- net DATA14: now also U?.16 (S14)
- net DATA15: now also U?.17 (S15)
- net DATA16: now also U?.1 (S0)
- net DATA17: now also U?.2 (S1)
- net DATA18: now also U?.3 (S2)
- net DATA19: now also U?.4 (S3)
- net DATA20: now also U?.5 (S4)
- net DATA21: now also U?.6 (S5)
- net DATA22: now also U?.7 (S6)
- net DATA23: now also U?.8 (S7)
- net DATA24: now also U?.9 (S8)
- net DATA25: now also U?.10 (S9)
- net DATA26: now also U?.11 (S10)
- net DATA27: now also U?.13 (S11)
- net DATA28: now also U?.14 (S12)
- net DATA29: now also U?.15 (S13)
- net DATA30: now also U?.16 (S14)
- net DATA31: now also U?.17 (S15)
- net DATAR: now also U?.19 (E1), U?.19 (E1)
- net GND: now also J?.1, J?.5, J?.9 (SHIELD), U?.12 (GND), U?.12 (GND)
- net RxIN: now also J?.4, J?.8
- net VCC: now also U?.24 (VCC), U?.24 (VCC)
- net nRxIN: now also J?.3, J?.7
- net A3: now reaches U?.11 ((PCINT21/OC0B/T1)PD5)
- net A3: now also U?.20 (A3), U?.20 (A3)
- net G: now reaches U?.12 ((PCINT22/OC0A/AIN0)PD6)
- net G: now also U?.18 (E0)
- net ~G: now reaches U?.13 ((PCINT23/AIN1)PD7)
- net ~G: now also U?.18 (E0)
- net A0: now reaches U?.4 ((PCINT18/INT0)PD2)
- net A0: now also U?.23 (A0), U?.23 (A0)
- net A1: now reaches U?.5 ((PCINT19/OC2B/INT1)PD3)
- net A1: now also U?.22 (A1), U?.22 (A1)
- net A2: now reaches U?.6 ((PCINT20/XCK/T0)PD4)
- net A2: now also U?.21 (A2), U?.21 (A2)
- no-connect marks 9 -> 11
Other:
- note added: "Line Decoder"
- note added: "RS-485 Tx"
- note removed: "RS-485 Decoder"
- moved on the sheet: J?, U?, U?A, U?B, U?C, U?D, U?E, U?F

Commit message: + Layout
Parts:
- J1, J2: renamed from J?; footprint (none) -> Connectors:RJ45_TRANSFO_ver2
- J10, J11, J12, J13, J14, J15, J16, J17, J18, J19, J20, J21, J22, J23, J24, J25, J26, J27, J28, J29, J3, J30, J31, J32, J33, J34, J4, J5, J6, J7, J8, J9: renamed from J?; footprint (none) -> Connectors_Terminal_Blocks:TerminalBlock_Pheonix_MPT-2.54mm_4pol
- U1: renamed from U?; footprint (none) -> Housings_DIP:DIP-14_W7.62mm_Socket_LongPads
- U2: renamed from U?; footprint DIL28 -> Housings_DIP:DIP-28_W7.62mm_Socket_LongPads
- U3: renamed from U?; footprint (none) -> Housings_DIP:DIP-16_W7.62mm_Socket_LongPads
- U4: renamed from U?; footprint (none) -> Housings_DIP:DIP-8_W7.62mm_Socket_LongPads
- U5, U6: renamed from U?; footprint (none) -> Housings_DIP:DIP-24_W7.62mm_Socket_LongPads
Connections:
- net at U2.1 ((PCINT14/~RESET~)PC6): now also U3.1; no longer U3.7
- net at U2.23 ((PCINT8/ADC0)PC0): now also U3.7; no longer U3.1
- net at U2.24 ((PCINT9/ADC1)PC1): now also U3.6; no longer U3.2
- net at U2.25 ((PCINT10/ADC2)PC2): now also U3.5; no longer U3.3
- net at U2.27 ((PCINT12/SDA/ADC4)PC4): now also U3.3; no longer U3.5
- net at U2.28 ((PCINT13/SCL/ADC5)PC5): now also U3.2; no longer U3.6
Other:
- moved on the sheet: U3
